Commit message: Add files via upload

File: ar10_description/urdf/ar10l.urdf (robot description, URDF)
Before this commit: robot ar10, 48 links, 47 joints
Links:
- link palm: geometry collision mesh filename=package://ar10_description/meshes/Palm -RIGHT.STL scale=.001 .001 .001; visual mesh filename=package://ar10_description/meshes/Palm-LEFT.STL scale=.001 .001 .001
Joints:
- joint ee1: origin xyz=-.005 0 -.02 rpy=0 0 0 -> xyz=.005 0 -.02 rpy=0 0 0
- joint ee2: origin xyz=-.005 0 -.02 rpy=0 0 0 -> xyz=.005 0 -.02 rpy=0 0 0
- joint ee3: origin xyz=-.005 0 -.02 rpy=0 0 0 -> xyz=.005 0 -.02 rpy=0 0 0
- joint ee4: origin xyz=-.005 0 -.02 rpy=0 0 0 -> xyz=.005 0 -.02 rpy=0 0 0
- joint rb10_to_palm: origin xyz=-.041 -.012 .022 rpy=0 -1.29 0 -> xyz=.041 -.012 .022 rpy=0 1.29 0
- joint rb1_to_palm: origin xyz=.0235 -.012 .08 -> xyz=-.0235 -.012 .08
- joint rb2_to_palm: origin xyz=.0105 -.012 .08 -> xyz=-.0105 -.012 .08
- joint rb3_to_palm: origin xyz=.0027 -.012 .09 -> xyz=-.0027 -.012 .09
- joint rb4_to_palm: origin xyz=-.011 -.012 .09 -> xyz=.011 -.012 .09
- joint rb5_to_palm: origin xyz=-.019 -.012 .1 -> xyz=.019 -.012 .1
- joint rb6_to_palm: origin xyz=-.032 -.012 .1 -> xyz=.032 -.012 .1
- joint rb7_to_palm: origin xyz=-.04 -.012 .095 -> xyz=.04 -.012 .095
- joint rb8_to_palm: origin xyz=-.053 -.012 .095 -> xyz=.053 -.012 .095
- joint rb9_to_palm: origin xyz=-.039 -.012 .0295 rpy=0 -1.29 0 -> xyz=.039 -.012 .0295 rpy=0 1.29 0
- joint servo0: axis -1 0 0 -> 1 0 0; origin xyz=-.0015 0 0 rpy= -1.57 0 0  -> xyz=.0015 0 0 rpy= -1.57 0 3.14 
- joint servo2: origin xyz=-.002 0 0 rpy=3.14 0 0 -> xyz=.002 0 0 rpy=3.14 0 0
- joint servo2m: origin xyz=.002 0 0 rpy=3.14 0 0 -> xyz=-.002 0 0 rpy=3.14 0 0
- joint servo3: origin xyz=.001 0 -.045 rpy=0 0 0 -> xyz=-.001 0 -.045 rpy=0 0 0
- joint servo3m: origin xyz=-.001 0 -.045 rpy=0 0 0 -> xyz=.001 0 -.045 rpy=0 0 0
- joint servo4: origin xyz=-.002 0 0 rpy=3.14 0 0 -> xyz=.002 0 0 rpy=3.14 0 0
- joint servo4m: origin xyz=.002 0 0 rpy=3.14 0 0 -> xyz=-.002 0 0 rpy=3.14 0 0
- joint servo5: origin xyz=.001 0 -.045 rpy=0 0 0 -> xyz=-.001 0 -.045 rpy=0 0 0
- joint servo5m: origin xyz=-.001 0 -.045 rpy=0 0 0 -> xyz=.001 0 -.045 rpy=0 0 0
- joint servo6: origin xyz=-.002 0 0 rpy=3.14 0 0 -> xyz=.002 0 0 rpy=3.14 0 0
- joint servo6m: origin xyz=.002 0 0 rpy=3.14 0 0 -> xyz=-.002 0 0 rpy=3.14 0 0
- joint servo7: origin xyz=.001 0 -.045 rpy=0 0 0 -> xyz=-.001 0 -.045 rpy=0 0 0
- joint servo7m: origin xyz=-.001 0 -.045 rpy=0 0 0 -> xyz=.001 0 -.045 rpy=0 0 0
- joint servo8: origin xyz=-.002 0 0 rpy=3.14 0 0 -> xyz=.002 0 0 rpy=3.14 0 0
- joint servo8m: origin xyz=.002 0 0 rpy=3.14 0 0 -> xyz=-.002 0 0 rpy=3.14 0 0
- joint servo9: origin xyz=.001 0 -.045 rpy=0 0 0 -> xyz=-.001 0 -.045 rpy=0 0 0
- joint servo9m: origin xyz=-.001 0 -.045 rpy=0 0 0 -> xyz=.001 0 -.045 rpy=0 0 0
- joint tip1: origin xyz=-.001 0 -.03 rpy=0 0 0 -> xyz=.001 0 -.03 rpy=0 0 0
- joint tip1b: origin xyz=.001 0 -.03 rpy=0 0 0 -> xyz=-.001 0 -.03 rpy=0 0 0
- joint tip2: origin xyz=-.001 0 -.03 rpy=0 0 0 -> xyz=.001 0 -.03 rpy=0 0 0
- joint tip2b: origin xyz=.001 0 -.03 rpy=0 0 0 -> xyz=-.001 0 -.03 rpy=0 0 0
- joint tip3: origin xyz=-.001 0 -.03 rpy=0 0 0 -> xyz=.001 0 -.03 rpy=0 0 0
- joint tip3b: origin xyz=.001 0 -.03 rpy=0 0 0 -> xyz=-.001 0 -.03 rpy=0 0 0
- joint tip4: origin xyz=-.001 0 -.03 rpy=0 0 0 -> xyz=.001 0 -.03 rpy=0 0 0
- joint tip4b: origin xyz=.001 0 -.03 rpy=0 0 0 -> xyz=-.001 0 -.03 rpy=0 0 0

File: ar10_description/urdf/ar10mesh.urdf (robot description, URDF)
Before this commit: robot ar10, 48 links, 47 joints
Joints:
- joint servo1: limit lower=0.34 upper=1.5 effort=1000.0 velocity=0.5 -> lower=0.0 upper=1.5 effort=1000.0 velocity=0.5
